File: MRCS-cpNode-ProMini v3.1a.brd (EAGLE design)
At the start: 99.8 x 68.8 mm, 59 parts, among them CON1 0.100, CON2 0.100, CON3 0.100, CON4 0.100, CON5 0.100, CON6 0.100, J1 0.100, J2 0.100, J3 2.1mm, P1 CA CC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

Commit message: changed value of pull down to 1K, moved Auto RTS resistor
The best value or the pull down on D13 (R1) is 1K, not 2.2K, mask adjusted.  Moved the autoRTS resistor (R2) so it's easier to change.
Parts:
- R3: value 2k2 -> 1K
- moved R1 19.1 mm to (17.1, 14.0)
- moved U$1 7.73 mm to (25.4, -10.2)
- moved C2 3.81 mm to (37.5, 12.7)
- moved C5 2.84 mm to (21.6, 12.7)
- moved D1 2.54 mm to (14.0, 15.2)
- moved U2 2.54 mm to (29.2, 12.7)
Routing:
- net N$52: track 33.3 -> 25.3 mm
- net VCC: track 284.6 -> 282.6 mm
- net GND: track 17.4 -> 15.4 mm
- net N$38: track 4.07 -> 5.50 mm
- net TXEN: track 30.6 -> 29.4 mm
- net TX: track 124.9 -> 125.7 mm
Other:
- board text added: "2021.12"
- board text added: "v3.1a"
- board text removed: "2021.06"
- board text removed: "v3.1"
